Commit message: commit

File: install/four_wheel_description/share/four_wheel_description/model/four_rover_main.gazebo.xacro (robot description, xacro)
@@ -1,29 +1,4 @@
 <?xml version="1.0"?>
 <robot>
-    <gazebo reference="base_link">
-        <mu1>0.2</mu1>
-        <mu2>0.2</mu2>
-        <material>Gazebo/Red</material>
-    </gazebo>
-    <gazebo reference="d1_wheel_link">
-        <mu1>0.2</mu1>
-        <mu2>0.2</mu2>
-        <material>Gazebo/Yellow</material>
-    </gazebo>
-    <gazebo reference="d2_wheel_link">
-        <mu1>0.2</mu1>
-        <mu2>0.2</mu2>
-        <material>Gazebo/Yellow</material>
-    </gazebo>
-    <gazebo reference="caster1_link">
-        <mu1>0.000002</mu1>
-        <mu2>0.000002</mu2>
-        <material>Gazebo/Blue</material>
-    </gazebo>
-    <gazebo reference="caster2_link">
-        <mu1>0.000002</mu1>
-        <mu2>0.000002</mu2>
-        <material>Gazebo/Blue</material>
-    </gazebo>
     <gazebo>
         <plugin filename="gz-sim-diff-drive-system" name="gz::sim::systems::DiffDrive">

File: install/four_wheel_description/share/four_wheel_description/model/four_rover_main.xacro (robot description, xacro)
@@ -24,5 +24,4 @@
     <xacro:property name="Iz_wheel" value="${0.5*m2*radius*radius}"/>
     <xacro:property name="I_wheel" value="${(1.0/12.0)*m2*(3.0*radius*radius+d*d)}"/>
-    <xacro:include filename="$(find four_wheel_description)/model/parts/camera/camera.xacro" />
     <xacro:macro name="inertia_body">
         <inertial>
@@ -39,118 +38,8 @@
         </inertial>
     </xacro:macro>
+    <xacro:include filename="$(find four_wheel_description)/model/parts/base/base_link.xacro"/>
+    <xacro:include filename="$(find four_wheel_description)/model/parts/camera/camera.xacro" />
+    <!-- <xacro:include filename="$(find four_wheel_description)/model/parts/lidar/lidar.xacro"/> -->
+    <xacro:include filename="$(find four_wheel_description)/model/parts/wheels/wheels.xacro"/>
     <xacro:include filename="$(find four_wheel_description)/model/four_rover_main.gazebo.xacro" />
-    <!-- Links and joints -->
-    <link name="base_footprint"> </link>
-    <joint name="base_link_joint" type="fixed">
-        <parent link="base_footprint"/>
-        <child link="base_link"/>
-    </joint>
-    <link name="base_link">
-        <visual>
-            <origin xyz="0 0 ${s1}" rpy="0 0 0"/>
-            <geometry>
-                <box size="${length} ${breadth} ${height}"/>
-            </geometry>
-        </visual>
-        <collision>
-            <origin xyz="0 0 ${s1}" rpy="0 0 0"/>
-            <geometry>
-                <box size="${length} ${breadth} ${height}"/>
-            </geometry>
-        </collision>
-        <xacro:inertia_body />
-    </link>
-    <joint name="d1_wheel_joint" type="continuous">
-        <parent link="base_link"/>
-        <child link="d1_wheel_link"/>
-        <origin xyz="${-s2} ${-s4} ${radius}" rpy="0 0 0" />
-        <axis xyz="0 1 0" />
-        <limit effort="50000" velocity="10"/>
-        <dynamics damping="1.0" friction="1.0" />
-    </joint>
-    <link name="d1_wheel_link">
-        <visual>
-            <origin xyz="0 0.0 0.0" rpy="1.570795 0.0 0.0"/>
-            <geometry>
-                <cylinder radius="${radius}" length="${d}"/>
-            </geometry>
-        </visual>
-        <collision>
-            <origin xyz="0 0.0 0.0" rpy="1.570795 0.0 0.0"/>
-            <geometry>
-                <cylinder radius="${radius}" length="${d}"/>
-            </geometry>
-        </collision>
-        <xacro:inertia_wheel />
-    </link>
-    <joint name="d2_wheel_joint" type="continuous">
-        <parent link="base_link"/>
-        <child link="d2_wheel_link"/>
-        <origin xyz="${-s2} ${s4} ${radius}" rpy="0.0 0.0 0.0"/>
-        <axis xyz="0 1 0"/>
-        <limit effort="50000" velocity="10"/>
-        <dynamics damping="1.0" friction="1.0" />
-    </joint>
-    <link name="d2_wheel_link">
-        <visual>
-            <origin xyz="0 0.0 0.0" rpy="1.570795 0.0 0.0"/>
-            <geometry>
-                <cylinder radius="${radius}" length="${d}"/>
-            </geometry>
-        </visual>
-        <collision>
-            <origin xyz="0 0.0 0.0" rpy="1.570795 0.0 0.0"/>
-            <geometry>
-                <cylinder radius="${radius}" length="${d}"/>
-            </geometry>
-        </collision>
-        <xacro:inertia_wheel />
-    </link>
-    <!-- Caster wheels  -->
-     <link name="caster1_link">
-        <visual>
-            <origin xyz="0 0 0" rpy="1.570795 0 0"/>
-            <geometry>
-                <cylinder radius="${radius}" length="${d}"/>
-            </geometry>
-        </visual>
-        <collision>
-            <origin xyz="0 0 0" rpy="1.570795 0 0"/>
-            <geometry>
-                <cylinder radius="${radius}" length="${d}"/>
-            </geometry>
-        </collision>
-        <xacro:inertia_wheel />
-    </link>
-    <joint name="caster1_joint" type="fixed">
-        <parent link="base_link"/>
-        <child link="caster1_link"/>
-        <origin xyz="${s2} ${-s4} ${radius}" rpy="0 0 0" />
-        <axis xyz="0 1 0"/>
-        <limit effort="50000" velocity="10"/>
-        <dynamics damping="1.0" friction="1.0" />
-    </joint>
-    <link name="caster2_link">
-        <visual>
-            <origin xyz="0 0 0" rpy="1.570795 0 0"/>
-            <geometry>
-                <cylinder radius="${radius}" length="${d}"/>
-            </geometry>
-        </visual>
-        <collision>
-            <origin xyz="0 0 0" rpy="1.570795 0 0"/>
-            <geometry>
-                <cylinder radius="${radius}" length="${d}"/>
-            </geometry>
-        </collision>
-        <xacro:inertia_wheel />
-    </link>
-    <joint name="caster2_joint" type="fixed">
-        <parent link="base_link"/>
-        <child link="caster2_link"/>
-        <origin xyz="${s2} ${s4} ${radius}" rpy="0 0 0" />
-        <axis xyz="0 1 0"/>
-        <limit effort="50000" velocity="10"/>
-        <dynamics damping="1.0" friction="1.0" />
-    </joint>
 </robot>

File: install/four_wheel_description/share/four_wheel_description/model/parts/base/base_link.gazebo.xacro (robot description, xacro)
@@ -1,3 +1,8 @@
 <?xml version="1.0"?>
 <robot xmlns:xacro="http://www.ros.org/wiki/xacro">
+    <gazebo reference="base_link">
+        <mu1>0.2</mu1>
+        <mu2>0.2</mu2>
+        <material>Gazebo/Red</material>
+    </gazebo>
 </robot>

File: install/four_wheel_description/share/four_wheel_description/model/parts/base/base_link.xacro (robot description, xacro)
@@ -1,4 +1,24 @@
 <?xml version="1.0"?>
 <robot xmlns:xacro="http://www.ros.org/wiki/xacro">
+    <link name="base_footprint"> </link>
+    <joint name="base_link_joint" type="fixed">
+        <parent link="base_footprint"/>
+        <child link="base_link"/>
+    </joint>
+    <link name="base_link">
+        <visual>
+            <origin xyz="0 0 ${s1}" rpy="0 0 0"/>
+            <geometry>
+                <box size="${length} ${breadth} ${height}"/>
+            </geometry>
+        </visual>
+        <collision>
+            <origin xyz="0 0 ${s1}" rpy="0 0 0"/>
+            <geometry>
+                <box size="${length} ${breadth} ${height}"/>
+            </geometry>
+        </collision>
+        <xacro:inertia_body />
+    </link>
     <xacro:include filename="$(find four_wheel_description)/model/parts/base/base_link.gazebo.xacro" />
 </robot>

File: install/four_wheel_description/share/four_wheel_description/model/parts/wheels/wheels.gazebo.xacro (robot description, xacro)
@@ -1,3 +1,23 @@
 <?xml version="1.0"?>
 <robot xmlns:xacro="http://www.ros.org/wiki/xacro">
+    <gazebo reference="d1_wheel_link">
+        <mu1>0.2</mu1>
+        <mu2>0.2</mu2>
+        <material>Gazebo/Yellow</material>
+    </gazebo>
+    <gazebo reference="d2_wheel_link">
+        <mu1>0.2</mu1>
+        <mu2>0.2</mu2>
+        <material>Gazebo/Yellow</material>
+    </gazebo>
+    <gazebo reference="caster1_link">
+        <mu1>0.000002</mu1>
+        <mu2>0.000002</mu2>
+        <material>Gazebo/Blue</material>
+    </gazebo>
+    <gazebo reference="caster2_link">
+        <mu1>0.000002</mu1>
+        <mu2>0.000002</mu2>
+        <material>Gazebo/Blue</material>
+    </gazebo>
 </robot>

File: install/four_wheel_description/share/four_wheel_description/model/parts/wheels/wheels.xacro (robot description, xacro)
@@ -1,4 +1,97 @@
 <?xml version="1.0"?>
 <robot xmlns:xacro="http://www.ros.org/wiki/xacro">
+    <joint name="d1_wheel_joint" type="continuous">
+        <parent link="base_link"/>
+        <child link="d1_wheel_link"/>
+        <origin xyz="${-s2} ${-s4} ${radius}" rpy="0 0 0" />
+        <axis xyz="0 1 0" />
+        <limit effort="50000" velocity="10"/>
+        <dynamics damping="1.0" friction="1.0" />
+    </joint>
+    <link name="d1_wheel_link">
+        <visual>
+            <origin xyz="0 0.0 0.0" rpy="1.570795 0.0 0.0"/>
+            <geometry>
+                <cylinder radius="${radius}" length="${d}"/>
+            </geometry>
+        </visual>
+        <collision>
+            <origin xyz="0 0.0 0.0" rpy="1.570795 0.0 0.0"/>
+            <geometry>
+                <cylinder radius="${radius}" length="${d}"/>
+            </geometry>
+        </collision>
+        <xacro:inertia_wheel />
+    </link>
+    <joint name="d2_wheel_joint" type="continuous">
+        <parent link="base_link"/>
+        <child link="d2_wheel_link"/>
+        <origin xyz="${-s2} ${s4} ${radius}" rpy="0.0 0.0 0.0"/>
+        <axis xyz="0 1 0"/>
+        <limit effort="50000" velocity="10"/>
+        <dynamics damping="1.0" friction="1.0" />
+    </joint>
+    <link name="d2_wheel_link">
+        <visual>
+            <origin xyz="0 0.0 0.0" rpy="1.570795 0.0 0.0"/>
+            <geometry>
+                <cylinder radius="${radius}" length="${d}"/>
+            </geometry>
+        </visual>
+        <collision>
+            <origin xyz="0 0.0 0.0" rpy="1.570795 0.0 0.0"/>
+            <geometry>
+                <cylinder radius="${radius}" length="${d}"/>
+            </geometry>
+        </collision>
+        <xacro:inertia_wheel />
+    </link>
+    <!-- Caster wheels  -->
+     <link name="caster1_link">
+        <visual>
+            <origin xyz="0 0 0" rpy="1.570795 0 0"/>
+            <geometry>
+                <cylinder radius="${radius}" length="${d}"/>
+            </geometry>
+        </visual>
+        <collision>
+            <origin xyz="0 0 0" rpy="1.570795 0 0"/>
+            <geometry>
+                <cylinder radius="${radius}" length="${d}"/>
+            </geometry>
+        </collision>
+        <xacro:inertia_wheel />
+    </link>
+    <joint name="caster1_joint" type="fixed">
+        <parent link="base_link"/>
+        <child link="caster1_link"/>
+        <origin xyz="${s2} ${-s4} ${radius}" rpy="0 0 0" />
+        <axis xyz="0 1 0"/>
+        <limit effort="50000" velocity="10"/>
+        <dynamics damping="1.0" friction="1.0" />
+    </joint>
+    <link name="caster2_link">
+        <visual>
+            <origin xyz="0 0 0" rpy="1.570795 0 0"/>
+            <geometry>
+                <cylinder radius="${radius}" length="${d}"/>
+            </geometry>
+        </visual>
+        <collision>
+            <origin xyz="0 0 0" rpy="1.570795 0 0"/>
+            <geometry>
+                <cylinder radius="${radius}" length="${d}"/>
+            </geometry>
+        </collision>
+        <xacro:inertia_wheel />
+    </link>
+    <joint name="caster2_joint" type="fixed">
+        <parent link="base_link"/>
+        <child link="caster2_link"/>
+        <origin xyz="${s2} ${s4} ${radius}" rpy="0 0 0" />
+        <axis xyz="0 1 0"/>
+        <limit effort="50000" velocity="10"/>
+        <dynamics damping="1.0" friction="1.0" />
+    </joint>
     <xacro:include filename="$(find four_wheel_description)/model/parts/wheels/wheels.gazebo.xacro" />
 </robot>

File: src/four_wheel_description/model/four_rover_main.xacro (robot description, xacro)
@@ -38,8 +38,8 @@
         </inertial>
     </xacro:macro>
+    <xacro:include filename="$(find four_wheel_description)/model/parts/base/base_link.xacro"/>
+    <xacro:include filename="$(find four_wheel_description)/model/parts/camera/camera.xacro" />
+    <!-- <xacro:include filename="$(find four_wheel_description)/model/parts/lidar/lidar.xacro"/> -->
+    <xacro:include filename="$(find four_wheel_description)/model/parts/wheels/wheels.xacro"/>
     <xacro:include filename="$(find four_wheel_description)/model/four_rover_main.gazebo.xacro" />
-    <xacro:include filename="$(find four_wheel_description)/model/parts/base/base_link.xacro"/>
-    <xacro:include filename="$(find four_wheel_description)/model/parts/wheels/wheels.xacro"/>
-    <!-- <xacro:include filename="$(find four_wheel_description)/model/parts/lidar/lidar.xacro"/> -->
-    <xacro:include filename="$(find four_wheel_description)/model/parts/camera/camera.xacro" />
 </robot>
