Commit message: Updated movement and odometry fixes

File: src/four_wheel_description/model/four_rover_main.gazebo.xacro (robot description, xacro)
@@ -1,23 +1,27 @@
 <?xml version="1.0"?>
 <robot>
-    <gazebo>
-        <plugin filename="gz-sim-diff-drive-system" name="gz::sim::systems::DiffDrive">
-            <right_joint>d1_wheel_joint</right_joint>
-            <left_joint>d2_wheel_joint</left_joint>
-            <wheel_seperation>${2*s4}</wheel_seperation>
-            <wheel_diameter>${2*radius}</wheel_diameter>
-            <max_linear_acceleration>10</max_linear_acceleration>
-            <topic>cmd_vel</topic>
-            <tf_topic>/tf</tf_topic>
-            <odom_topic>odom</odom_topic>
-            <frame_id>odom</frame_id>
-            <child_frame_id>base_footprint</child_frame_id>
-            <odom_publisher_frequency>30</odom_publisher_frequency>
-        </plugin>
-        <plugin filename="gz-sim-joint-state-publisher-system" name="gz::sim::systems::JointStatePublisher">
-            <topic>joint_states</topic>
-            <joint_name>d1_wheel_joint</joint_name>
-            <joint_name>d2_wheel_joint</joint_name>
-        </plugin>
-    </gazebo>
+      <gazebo>
+            <plugin filename="gz-sim-diff-drive-system"
+                    name="gz::sim::systems::DiffDrive">
+              <left_joint>left_wheel_joint</left_joint>
+              <right_joint>right_wheel_joint</right_joint>
+              <wheel_separation>${2*s4}</wheel_separation>
+              <wheel_radius>${radius}</wheel_radius>
+              <odom_publish_frequency>20</odom_publish_frequency>
+              <topic>cmd_vel</topic>
+              <odom_topic>odom</odom_topic>
+              <tf_topic>tf</tf_topic>
+              <frame_id>odom</frame_id>
+              <child_frame_id>base_footprint</child_frame_id>
+              <max_linear_acceleration>1.0</max_linear_acceleration>
+            </plugin>
+  </gazebo>
+  <gazebo>
+    <plugin filename="gz-sim-joint-state-publisher-system"
+            name="gz::sim::systems::JointStatePublisher">
+      <joint_name>left_wheel_joint</joint_name>
+      <joint_name>right_wheel_joint</joint_name>
+      <topic>joint_states</topic>
+    </plugin>
+  </gazebo>
 </robot>

File: src/four_wheel_description/model/parts/wheels/wheels.xacro (robot description, xacro)
@@ -1,13 +1,5 @@
 <?xml version="1.0"?>
 <robot xmlns:xacro="http://www.ros.org/wiki/xacro">
-    <joint name="d1_wheel_joint" type="continuous">
-        <parent link="base_link"/>
-        <child link="d1_wheel_link"/>
-        <origin xyz="${-s2} ${-s4} ${radius}" rpy="0 0 0" />
-        <axis xyz="0 1 0" />
-        <limit effort="50000" velocity="10"/>
-        <dynamics damping="1.0" friction="1.0" />
-    </joint>
-    <link name="d1_wheel_link">
+    <link name="left_wheel_link">
         <visual>
             <origin xyz="0 0.0 0.0" rpy="1.570795 0.0 0.0"/>
@@ -24,13 +16,13 @@
         <xacro:inertia_wheel />
     </link>
-    <joint name="d2_wheel_joint" type="continuous">
+    <joint name="left_wheel_joint" type="continuous">
         <parent link="base_link"/>
-        <child link="d2_wheel_link"/>
-        <origin xyz="${-s2} ${s4} ${radius}" rpy="0.0 0.0 0.0"/>
-        <axis xyz="0 1 0"/>
+        <child link="left_wheel_link"/>
+        <origin xyz="${-s2} ${-s4} ${radius}" rpy="0 0 0" />
+        <axis xyz="0 1 0" />
         <limit effort="50000" velocity="10"/>
         <dynamics damping="1.0" friction="1.0" />
     </joint>
-    <link name="d2_wheel_link">
+    <link name="right_wheel_link">
         <visual>
             <origin xyz="0 0.0 0.0" rpy="1.570795 0.0 0.0"/>
@@ -47,4 +39,12 @@
         <xacro:inertia_wheel />
     </link>
+    <joint name="right_wheel_joint" type="continuous">
+        <parent link="base_link"/>
+        <child link="right_wheel_link"/>
+        <origin xyz="${-s2} ${s4} ${radius}" rpy="0.0 0.0 0.0"/>
+        <axis xyz="0 1 0"/>
+        <limit effort="50000" velocity="10"/>
+        <dynamics damping="1.0" friction="1.0" />
+    </joint>
     <!-- Caster wheels  -->
      <link name="caster1_link">
